File: ElmerFEM Test/ElmerFEM Test.kicad_sch (KiCad schematic)
At the start: 0 parts

Commit message: Elmer FEM Testing
I have a skeleton of a process to get the PCB into Elmer. I just need to refine the proces, get a simulation to converge and then write an automation script for it
I imagine the type and quality of solver will depend on the minimum geometry of the circuit.
Parts:
- added J1, J2, J3, J4: Conn_01x01, Connector:Banana_Jack_1Pin, symbol Connector_Generic:Conn_01x01
Connections:
- new net: J2.1 (Pin_1), J4.1 (Pin_1)
- new net: J1.1 (Pin_1), J3.1 (Pin_1)
