File: ElmerFEM_Test/ElmerFEM Test.kicad_pcb (KiCad board)
At the start: 4 copper layers, 53.3 x 40.6 mm, 4 parts, among them J1 Conn_01x01, J2 Conn_01x01, J3 Conn_01x01, J4 Conn_01x01

Commit message: Stable Release
- Minimally functional automated solver
Parts:
- added J5: Barrel_Jack, Battery:BatteryHolder_Keystone_103_1x20mm, F.Cu at (147.3, 85.4)
Routing:
- net /Test: track 0.00 -> 94.4 mm
Other:
- board size 53.3 x 40.6 mm -> 88.9 x 40.6 mm
