File: ElmerFEM_Test/ElmerFEM Test.kicad_sch (KiCad schematic)
At the start: 4 parts, among them J1 Conn_01x01, J2 Conn_01x01, J3 Conn_01x01, J4 Conn_01x01

Commit message: Stable Release
- Minimally functional automated solver
Parts:
- added J5: Barrel_Jack, Battery:BatteryHolder_Keystone_103_1x20mm, symbol Connector:Barrel_Jack
- J1: CCSIM.1 (none) -> 5A
- J2: CCSIM.1 (none) -> 5V
- J3: CCSIM.1 (none) -> -4.9A
- J4: CCSIM.1 (none) -> -0.1A
Connections:
- new net Test: J5.1, J5.2
